File: KiCAD/Basilisk.kicad_sch (KiCad schematic)
At the start: 56 parts

Commit message: finish schematic?
Parts:
- removed D?: ESP, symbol Device:LED_Small
- removed R?: 270, symbol Device:R
- added C1, C2, C3: 0.1uf, Capacitor_SMD:C_0805_2012Metric, symbol Device:C_Small
- added U3: MLX90640, basilisk:TO292P930H600-4, symbol basilisk:MLX90640
- C10, C11, C12, C13, C14, C15, C16, C17, C4, C5, C6, C7, C8, C9: renamed from C?; footprint (none) -> Capacitor_SMD:C_0805_2012Metric
- D1, D2: renamed from D?; footprint (none) -> Diode_SMD:D_SMC
- D3, D4: renamed from D?; footprint (none) -> LED_SMD:LED_0805_2012Metric
- J1: renamed from J?; footprint (none) -> Connector_Molex:Molex_KK-396_A-41791-0004_1x04_P3.96mm_Vertical
- J2: renamed from J?; footprint (none) -> Connector_PinSocket_2.54mm:PinSocket_2x08_P2.54mm_Vertical
- J3: renamed from J?; footprint (none) -> Connector_BarrelJack:BarrelJack_Horizontal
- J4: renamed from J?; footprint (none) -> Connector_USB:USB_C_Receptacle_GCT_USB4085
- R1, R10, R11, R12, R13, R14, R15, R16, R17, R18, R19, R2, R20, R3, R4, R5, R6, R7, R8, R9: renamed from R?; footprint (none) -> Resistor_SMD:R_0805_2012Metric
- SW1, SW2: renamed from SW?; footprint (none) -> Button_Switch_SMD:SW_SPST_TL3342
- gave numbers to parts that had none: 10
Connections:
- net +3.3V: now also C1.1, C2.1, C3.1, U3.4 (VCC)
- net B.3: now also U2.23 (IO15); no longer U2.36 (IO22)
- net C.3: now also U2.24 (IO2); no longer U2.33 (IO21)
- net GND: now also C1.2, C2.2, C3.2, U3.2 (GND)
- net IO0: now also U5.12 (B8)
- net SCL: now also U2.36 (IO22), U3.1 (SCL)
- net SDA: now also U2.33 (IO21), U3.3 (SDA)
- removed net OE.3: U2.23 (IO15), U5.12 (B8)
Other:
- moved on the sheet: R1, R2, U1
